Commit message: fixed minor errors

File: Exoskeleton3DOF_URDFmodel/ExoskeletonURDFmodel.urdf (robot description, URDF)
Before this commit: robot exoskeletonURDFmodel_noHuman, 3 links, 2 joints
Links:
- link ExoLeftLeg: geometry collision mesh filename=package://Exoskeleton3DOF_URDFmodel/meshes/sim_leftleg_prt.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 scale=0.001 0.001 0.001; visual mesh filename=package://Exoskeleton3DOF_URDFmodel/meshes/sim_leftleg_prt.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 scale=0.001 0.001 0.001
- link ExoRightLeg: geometry collision mesh filename=package://Exoskeleton3DOF_URDFmodel/meshes/sim_rightleg_prt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 scale=0.001 0.001 0.001; visual mesh filename=package://Exoskeleton3DOF_URDFmodel/meshes/sim_rightleg_prt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 scale=0.001 0.001 0.001
- link ExoTorso: geometry collision mesh filename=package://Exoskeleton3DOF_URDFmodel/meshes/sim_torso_prt.stl scale=0.001 0.001 0.001; visual mesh filename=package://Exoskeleton3DOF_URDFmodel/meshes/sim_torso_prt.stl scale=0.001 0.001 0.001
